File: PCB/Saunasteuerung-ESP-Home/io-expander.kicad_sch (KiCad schematic)
At the start: 5 parts, among them U7 PCA9685PW_118, U8 MCP23017T-E_ML

Commit message: Added AD5593
Parts:
- added U4: AD5593R, Package_SO:TSSOP-16_4.4x5mm_P0.65mm, symbol Analog:AD5593R
Changed lines of the file:
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@@
 (kicad_sch
-	(version 20231120)
+	(version 20250114)
 	(generator "eeschema")
-	(generator_version "8.0")
+	(generator_version "9.0")
 	(paper "A4")
 	(junction
@@
 					(unit 1)
 				)
+			)
+		)
+	)
+	(symbol
+		(lib_id "Analog:AD5593R")
+		(at 97.79 154.94 0)
+		(unit 1)
+		(exclude_from_sim no)
+		(in_bom yes)
+		(on_board yes)
+		(dnp no)
+		(fields_autoplaced yes)
+		(property "Reference" "U4"
+			(at 99.9333 168.91 0)
+			(effects
+				(font
+					(size 1.27 1.27)
+				)
+				(justify left)
+			)
+		)
+		(property "Value" "AD5593R"
+			(at 99.9333 171.45 0)
+			(effects
+				(font
+					(size 1.27 1.27)
+				)
+				(justify left)
+			)
+		)
+		(property "Footprint" "Package_SO:TSSOP-16_4.4x5mm_P0.65mm"
+			(at 123.19 167.64 0)
+			(effects
+				(font
+					(size 1.27 1.27)
+					(italic yes)
+				)
+				(hide yes)
+			)
+		)
+		(property "Datasheet" "https://www.analog.com/media/en/technical-documentation/data-sheets/AD5593R.pdf"
+			(at 97.79 160.02 0)
+			(effects
+				(font
+					(size 1.27 1.27)
+				)
+				(hide yes)
+			)
+		)
+		(property "Description" "8-channel 12bits configurable ADC/DAC/GPIO Internal Reference, I2C interface Integrated temperature sensor,Single Supply, TSSOP-16"
+			(at 97.79 154.94 0)
+			(effects
+				(font
+					(size 1.27 1.27)
+				)
+				(hide yes)
+			)
+		)
+		(pin "4"
+		)
+		(pin "6"
+		)
+		(pin "10"
+		)
+		(pin "1"
+		)
+		(pin "11"
+		)
+		(pin "12"
+		)
+		(pin "14"
+		)
+		(pin "16"
+		)
+		(pin "8"
+		)
+		(pin "2"
+		)
+		(pin "3"
+		)
+		(pin "15"
+		)
+		(pin "9"
+		)
+		(pin "5"
+		)
+		(pin "7"
+		)
+		(pin "13"
+		)
+		(instances
+			(project ""
+				(path "/c2709fca-2df2-4b64-83dc-e0d31f28d840/443e1443-1d33-4007-83fb-6df627e1fa6b"
+					(reference "U4")
+					(unit 1)
+				)

Commit message: V2.0 push
Parts:
- removed R25, R26, R27: 10k, Resistor_SMD:R_0603_1608Metric, symbol Device:R_Small
- removed U4: AD5593R, Package_SO:TSSOP-16_4.4x5mm_P0.65mm, symbol Analog:AD5593R
- removed U7: PCA9685PW_118, Snapeda:PCA9685PW_118_SOP65P640X110-28N, symbol Snapeda:PCA9685PW_118
- removed U8: MCP23017T-E_ML, Snapeda:MCP23017T-E_ML_QFN65P600X600X100-29N, symbol Snapeda:MCP23017T-E_ML
Connections:
- no-connect marks 23 -> 0
