File: PCB/Saunasteuerung-ESP-Home/Saunasteuerung-ESP-Home.kicad_pcb (KiCad board)
At the start: 2 copper layers, 245 x 110 mm, 87 parts, among them J1 HB9500M-9.5-6P, J2 HB9500M-9.5-6P, J3 HB9500M-9.5-6P, J4 HB9500M-9.5-3P, J5 I2C, J6 Nextion Display, J7 WS2812, J8 696106003002, K1 RAYEX-L90, K2 RAYEX-L90, K3 RAYEX-L90, K4 SANYOU_SRD_Form_C, K5 SANYOU_SRD_Form_C, Q1 S8550, Q10 2N7002, Q2 S8550, Q3 S8550, Q4 IRLZ34N, Q5 2N222, Q6 2N222, Q7 IRLZ34N, Q8 IRLZ34N, Q9 IRLZ34N, U1 FODM217A, U2 FODM217A, U3 FODM217A, U5 DS18B20, U6 MOUDLE-SEEEDUINO-XIAO-ESP32C3, U7 PCA9685PW_118, U8 MCP23017T-E_ML, X1 Sensors, X2 LED's

Commit message: V2.0 push
Parts:
- removed D16: LED, LED_SMD:LED_0603_1608Metric
- removed FL1: Filter_EMI_CommonMode, Inductor_THT:L_CommonMode_PulseElectronics_PH9455x105NL_1
- removed H1: WIZ850IO, Snapeda:WIZ850IO_WIZ850IO
- removed H4, H7: MountingHole_Pad, MountingHole:MountingHole_3.2mm_M3_DIN965_Pad_TopBottom
- removed J4: HB9500M-9.5-3P, Samacsys:HB9500M953P
- removed J6: Nextion Display, Connector_JST:JST_XH_B4B-XH-A_1x04_P2.50mm_Vertical
- removed U6: MOUDLE-SEEEDUINO-XIAO-ESP32C3, RF_Module:MCU_Seeed_ESP32C3
- removed U7: PCA9685PW_118, Snapeda:PCA9685PW_118_SOP65P640X110-28N
- removed U8: MCP23017T-E_ML, Snapeda:MCP23017T-E_ML_QFN65P600X600X100-29N
- added A1: ESP32-S3-ETH, ESP32-S3-ETH:ESP32-S3-ETH, F.Cu at (122.5, 90.1)
- added C3: 1uF, Capacitor_SMD:C_0603_1608Metric, F.Cu at (161.9, 136.2)
- added IC1: WS2811, WS2811:SO08-SKINNYPADS, F.Cu at (166.8, 133.3)
- added JP1: Low-Speed, Jumper:SolderJumper-2_P1.3mm_Open_TrianglePad1.0x1.5mm, F.Cu at (161.7, 127.9)
- added Q11: NTD5867NL, Package_TO_SOT_SMD:TO-252-2, F.Cu at (178.4, 140.9)
- added Q12: NTD5867NL, Package_TO_SOT_SMD:TO-252-2, F.Cu at (178.4, 161.6)
- added R28: 1k, Resistor_SMD:R_0603_1608Metric, F.Cu at (137.8, 121.3)
- added R29: 10k, Resistor_SMD:R_0603_1608Metric, F.Cu at (134.7, 121.3)
- added R30: 1k, Resistor_SMD:R_0603_1608Metric, F.Cu at (120.9, 128.1)
- added R31: 1k, Resistor_SMD:R_0603_1608Metric, F.Cu at (137.5, 128.1)
- added R32: 10k, Resistor_SMD:R_0603_1608Metric, F.Cu at (165.9, 151.4)
- added R33: 1k, Resistor_SMD:R_0603_1608Metric, F.Cu at (165.9, 154.8)
- added R34: 10k, Resistor_SMD:R_0603_1608Metric, F.Cu at (172.5, 146.6)
- added R35: 1k, Resistor_SMD:R_0603_1608Metric, F.Cu at (164.3, 165.3)
- added R36: 10k, Resistor_SMD:R_0603_1608Metric, F.Cu at (166.0, 161.8)
- added R37: 1k, Resistor_SMD:R_0603_1608Metric, F.Cu at (166.0, 165.3)
- added R38: 10k, Resistor_SMD:R_0603_1608Metric, F.Cu at (172.5, 157.0)
- added U10: FODM217A, Package_SO:SOP-4_4.4x2.6mm_P1.27mm, F.Cu at (128.5, 124.3)
- added U9: FODM217A, Package_SO:SOP-4_4.4x2.6mm_P1.27mm, F.Cu at (111.9, 124.3)
- D10: value LED -> 1N4148W; footprint LED_SMD:LED_0603_1608Metric -> Diode_SMD:D_SOD-123
- D7: value 1N4148W -> LED; footprint Diode_SMD:D_SOD-123 -> LED_SMD:LED_0603_1608Metric
- K4, K5: value SANYOU_SRD_Form_C -> G2RL-1-E; footprint Relay_THT:Relay_SPDT_SANYOU_SRD_Series_Form_C -> Relay_THT:Relay_SPDT_Omron_G2RL-1-E
- Q4, Q7, Q9: value IRLZ34N -> BSS214NW; footprint Package_TO_SOT_THT:TO-220-3_Vertical -> Package_TO_SOT_SMD:SOT-323_SC-70
- Q5, Q6: value 2N222 -> S8550; footprint Package_TO_SOT_THT:TO-92L -> Package_TO_SOT_SMD:SOT-23
- Q8: value IRLZ34N -> NTD5867NL; footprint Package_TO_SOT_THT:TO-220-3_Vertical -> Package_TO_SOT_SMD:TO-252-2
- R17, R24: value 1k -> 10k
- R21: value 1k -> 33
- R22: value 1k -> 100
- R25, R27: value 10k -> 1k
- moved R18 96.6 mm to (161.2, 83.8), turned to -90 degrees
- moved Q10 92.6 mm to (164.1, 83.7), turned to -90 degrees
- moved R24 84.9 mm to (165.9, 141.0)
- moved J5 82.6 mm to (90.4, 86.2)
- moved R22 80.9 mm to (161.9, 130.3), turned to 0 degrees
- moved LS1 79.4 mm to (173.5, 84.8), turned to 180 degrees
- moved R23 77.7 mm to (164.3, 144.4)
- moved Q9 76.1 mm to (169.7, 163.2), turned to 0 degrees
- moved D15 75.2 mm to (164.3, 161.8)
- moved D13 75.0 mm to (164.3, 141.0)
- moved D14 74.6 mm to (164.3, 151.4)
- moved Q7 73.8 mm to (169.8, 152.8), turned to 0 degrees
- moved Q4 73.8 mm to (169.8, 142.5), turned to 0 degrees
- moved R21 73.4 mm to (167.5, 127.4), turned to -90 degrees
- moved Q8 68.2 mm to (178.4, 151.1), turned to 0 degrees
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Connections:
- D10 pad 2: Net-(D10-A) -> GND
- D13 pad 1: GND -> Net-(D13-K)
- D13 pad 2: Net-(D13-A) -> +5V
- D14 pad 1: GND -> Net-(D14-K)
- D14 pad 2: Net-(D14-A) -> +5V
- D15 pad 1: GND -> Net-(D15-K)
- D15 pad 2: Net-(D15-A) -> +5V
- D7 pad 1: +5V -> GND
- D7 pad 2: Net-(D10-K) -> Net-(D7-A)
- D8 pad 1: +5V -> Net-(D8-K)
- D8 pad 2: Net-(D8-A) -> GND
- D9 pad 1: Net-(D8-A) -> GND
- H2 pad 1: GND -> unconnected-(H2-Pad1)
- H3 pad 1: GND -> unconnected-(H3-Pad1)
- H5 pad 1: GND -> unconnected-(H5-Pad1)
- H6 pad 1: GND -> unconnected-(H6-Pad1)
- J1 pad 2: Net-(J1-Pad2) -> L1
- J1 pad 3: L1 -> Net-(J1-Pad3)
- J3 pad 1: Net-(J3-Pad1) -> N
- J3 pad 2: Net-(J3-Pad2) -> N
- J3 pad 3: Net-(J3-Pad3) -> N
- J3 pad 4: N -> GND
- J3 pad 5: N -> GND
- J3 pad 6: N -> GND
- J5 pad 2: SCK -> SDA
- J5 pad 3: SDA -> SCK
- J8 pad 2: Net-(C2-Pad1) -> unconnected-(J8-Pad2)
- K1 pad 12: Net-(J1-Pad1) -> unconnected-(K1-Pad12)
- K1 pad 14: Net-(J1-Pad2) -> Net-(J1-Pad1)
- K2 pad 11A: Net-(J1-Pad6) -> Net-(J1-Pad4)
- K2 pad 11B: Net-(J1-Pad6) -> Net-(J1-Pad4)
- K2 pad 12: Net-(J1-Pad4) -> unconnected-(K2-Pad12)
- K2 pad 14: Net-(J1-Pad5) -> Net-(J1-Pad3)
- K3 pad 11A: Net-(J2-Pad3) -> Net-(J1-Pad6)
- K3 pad 11B: Net-(J2-Pad3) -> Net-(J1-Pad6)
- K3 pad 12: Net-(J2-Pad1) -> unconnected-(K3-Pad12)
- K3 pad 14: Net-(J2-Pad2) -> Net-(J1-Pad5)
- PS1 pad 1: Net-(PS1-AC1) -> unconnected-(J8-Pad2)
- PS1 pad 2: Net-(PS1-AC2) -> N
- Q4 pad 1: SIG-LED1 -> Net-(Q4-G)
- Q4 pad 2: LED1 -> GND
- Q4 pad 3: GND -> Net-(Q11-G)
- Q5 pad 1: GND -> Net-(Q5-B)
- Q5 pad 2: Net-(Q5-B) -> +5V
- Q5 pad 3: Net-(D10-K) -> Net-(D8-K)
- Q6 pad 1: GND -> Net-(Q6-B)
- Q6 pad 2: Net-(Q6-B) -> +5V
- Q6 pad 3: Net-(D8-A) -> Net-(D10-K)
- Q7 pad 1: SIG-LED2 -> Net-(Q7-G)
- Q7 pad 2: LED2 -> GND
- Q7 pad 3: GND -> Net-(Q7-D)
- Q8 pad 1: SIG-LED3 -> Net-(Q7-D)
- Q8 pad 2: LED3 -> LED2
- Q9 pad 1: SIG-LED4 -> Net-(Q9-G)
- Q9 pad 2: LED4 -> GND
- Q9 pad 3: GND -> Net-(Q12-G)
- R13 pad 1: SIG-RELAY4 -> +5V
- R13 pad 2: Net-(Q5-B) -> Net-(R13-Pad2)
- R14 pad 1: SIG-RELAY5 -> +5V
- R14 pad 2: Net-(Q6-B) -> Net-(R14-Pad2)
- R16 pad 1: Net-(D9-A) -> Net-(R16-Pad1)
- R16 pad 2: +5V -> Net-(Q5-B)
- R17 pad 1: Net-(D10-A) -> Net-(R16-Pad1)
- R21 pad 1: Net-(D13-A) -> WS2811-DIN
- R21 pad 2: SIG-LED1 -> Net-(IC1-DIN)
- R22 pad 1: Net-(D14-A) -> +5V
- R22 pad 2: SIG-LED2 -> Net-(IC1-VDD)
- R23 pad 1: Net-(D15-A) -> Net-(IC1-B)
- R23 pad 2: SIG-LED3 -> Net-(D13-K)
- R24 pad 1: Net-(D16-A) -> +5V
- R24 pad 2: SIG-LED4 -> Net-(Q4-G)
- R25 pad 1: Net-(U7-~OE) -> Net-(Q4-G)
- R25 pad 2: GND -> Net-(IC1-B)
- R26 pad 1: Net-(U7-A0) -> +5V
- R26 pad 2: GND -> Net-(Q11-G)
- R27 pad 2: GND -> Net-(D14-K)
- RV1 pad 1: Net-(C2-Pad1) -> unconnected-(J8-Pad2)
- X2 pad L1: LED1 -> +5V
- X2 pad L10: LED4 -> LED3
- X2 pad L2: Net-(X2-PadL2) -> WS2812
- X2 pad L3: Net-(X2-PadL2) -> GND
- X2 pad L4: LED2 -> LED1
- X2 pad L7: LED3 -> LED2
Routing:
- net GND: track 359.8 -> 160.1 mm, vias 24 -> 3
- net WS2812: track 0.00 -> 111.1 mm
- net SDA: track 132.8 -> 27.5 mm, vias 2 -> 0
- net SCK: track 128.6 -> 24.9 mm, vias 3 -> 0
- net WS2811-DIN: track 0.00 -> 102.2 mm
- net N: track 346.9 -> 258.9 mm
- net Net-(J1-Pad2): track 82.3 -> 0.00 mm
- net Net-(J3-Pad2): track 81.9 -> 0.00 mm
- net Net-(J1-Pad3): track 0.00 -> 76.4 mm
- net Thermo-Fuse1: track 145.1 -> 80.5 mm
- net MOSI: track 62.4 -> 0.00 mm, vias 1 -> 0
- net SCLK: track 57.5 -> 0.00 mm, vias 1 -> 0
- net Net-(J1-Pad4): track 56.9 -> 113.9 mm
- net Net-(J3-Pad1): track 56.5 -> 0.00 mm
- net Net-(J3-Pad3): track 56.4 -> 0.00 mm
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- added copper zone on B.Cu, net +5V
- added copper zone on F.Cu, net GND
- removed copper zone on F.Cu, net +5V
- removed copper zone on B.Cu, net GND
Other:
- board size 245 x 110 mm -> 180.9 x 110 mm
- board text added: "3.3V"
- board text added: "5V"
- board text added: "GND"
- board text added: "jse technolitrix 07.04.26"
- board text added: "max. 1A"
- board text removed: "LED4"
- board text removed: "NC-L1"
- board text removed: "NC-L2"
- board text removed: "NC-L3"
- board text removed: "Nextion Display"
- board text removed: "max. 2.5A"

Commit message: update
Parts:
- removed J5: I2C, Connector_JST:JST_XH_B4B-XH-A_1x04_P2.50mm_Vertical
- added J4: Frontpanel I/O, Connector_JST:JST_XH_B8B-XH-A_1x08_P2.50mm_Vertical, F.Cu at (135.0, 107.7)
- added J6: Frontpanel I2C, Connector_JST:JST_XH_B5B-XH-A_1x05_P2.50mm_Vertical, F.Cu at (109.1, 107.7)
- added JP2: selcect, Jumper:SolderJumper-2_P1.3mm_Open_TrianglePad1.0x1.5mm, F.Cu at (174.0, 114.4)
- added JP3: psu disable, Jumper:SolderJumper-2_P1.3mm_Bridged_Pad1.0x1.5mm, F.Cu at (88.5, 97.2)
- added R39: 10k, Resistor_SMD:R_0603_1608Metric, F.Cu at (113.6, 95.4)
- added R40: 10k, Resistor_SMD:R_0603_1608Metric, F.Cu at (111.1, 95.4)
- added R41: 33, Resistor_SMD:R_0603_1608Metric, F.Cu at (171.2, 110.8)
- added R42: 33, Resistor_SMD:R_0603_1608Metric, F.Cu at (105.6, 102.8)
- moved R15 14.0 mm to (136.4, 94.6), turned to -90 degrees
- moved H6 13.0 mm to (158.0, 163.0)
- moved D11 4.90 mm to (141.4, 108.2)
- moved R19 4.90 mm to (141.4, 104.7)
- moved R18 3.80 mm to (164.6, 82.1), turned to 180 degrees
- moved H3 3.00 mm to (158.0, 85.0)
- moved LS1 1.60 mm to (175.1, 84.8)
- moved Q10 1.23 mm to (164.6, 84.8)
- moved C1 0.81 mm to (90.0, 104.6)
Connections:
- A1 pad 1: unconnected-(A1-GPIO20-Pad1) -> GPIO20
- A1 pad 15: WS2812 -> ROT-CLK
- A1 pad 16: WS2811-DIN -> ROT-DT
- A1 pad 17: unconnected-(A1-GPIO35-Pad17) -> ROT-SW
- A1 pad 19: unconnected-(A1-GPIO34-Pad19) -> BTN-1
- A1 pad 2: unconnected-(A1-GPIO19-Pad2) -> GPIO19
- A1 pad 20: unconnected-(A1-GPIO33-Pad20) -> BTN-2
- A1 pad 25: unconnected-(A1-GPIO1-Pad25) -> WS2812-2
- A1 pad 4: unconnected-(A1-GPIO48-Pad4) -> WS2812-1
- A1 pad 5: unconnected-(A1-GPIO47-Pad5) -> WS2811-DIN
- C1 pad 1: GND -> +5V
- C1 pad 2: +5V -> GND
- J7 pad 2: WS2812 -> Net-(J7-Pin_2)
- PS1 pad 4: +5V -> Net-(JP3-A)
- X2 pad L2: WS2812 -> WS2812-1.1
Routing:
- net WS2812: track 111.1 -> 0.00 mm
- net +3.3V: track 19.0 -> 69.2 mm
- net WS2812-1: track 0.00 -> 49.8 mm, vias 0 -> 2
- net ROT-CLK: track 0.00 -> 41.7 mm
- net BTN-2: track 0.00 -> 40.9 mm
- net BTN-1: track 0.00 -> 40.9 mm
- net ROT-DT: track 0.00 -> 40.8 mm
- net ROT-SW: track 0.00 -> 39.8 mm
- net WS2811-DIN: track 102.2 -> 69.9 mm, vias 0 -> 2
- net GPIO20: track 0.00 -> 31.3 mm
- net GPIO19: track 0.00 -> 31.3 mm
- net Net-(J7-Pin_2): track 0.00 -> 23.2 mm
- net GND: track 160.1 -> 179.8 mm, vias 3 -> 11
- net SIG-RELAY5: track 38.5 -> 56.8 mm
- net WS2812-1.1: track 0.00 -> 18.0 mm
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Other:
- board text added: "Frontpanel I/O"
- board text added: "Frontpanel I2C"
- board text added: "PSU disable"
- board text removed: "I2C"
